File: hardware/thesis_kicad/thesis_kicad.sch (KiCad schematic (older format))
At the start: 5 parts, among them J1 EZR32LG330F256R60G_J101, U1 DHT22, U2 BH1750, U3 BMP280

Commit message: Update schematic with small fixes
Parts:
- added C? (x2): 100n, symbol Device:C
- added J?: USB_B_Micro, symbol Connector:USB_B_Micro
- added Q? (x3): Q_NMOS_DGS, symbol Device:Q_NMOS_DGS
- added R?: 10k, symbol Device:R
- added R? (x6): R, symbol Device:R
- added R? (x2): 4.7K, symbol Device:R
- added U?: TEN20-2410WIN, Converter_DCDC:Converter_DCDC_TRACO_TEN20-xxxx_THT, symbol Converter_DCDC:TEN20-2410WIN
Connections:
- wire segments 32 -> 67
Other:
- note added: "BATTERY"
- note added: "BH1750 VDD: 3V3"
- note added: "BMP280 VIN: 3V3"
- note added: "DHT22 VDD: 5V0"
- note added: "POWER"
- note removed: "POWER SIGNALS"

Commit message: Remove incorrect parts from schematic
Parts:
- removed C?: 100n, symbol Device:C
- removed J?: USB_B_Micro, symbol Connector:USB_B_Micro
- removed Q? (x3): Q_NMOS_DGS, symbol Device:Q_NMOS_DGS
- removed R? (x6): R, symbol Device:R
- removed U3: BMP280, symbol thesisLib:BMP280
- removed U?: TEN20-2410WIN, Converter_DCDC:Converter_DCDC_TRACO_TEN20-xxxx_THT, symbol Converter_DCDC:TEN20-2410WIN
- added U?: BMP280, Package_LGA:Bosch_LGA-8_2x2.5mm_P0.65mm_ClockwisePinNumbering, symbol Sensor_Pressure:BMP280
Connections:
- net labels added: +5V, 5V0
- wire segments 67 -> 37
Other:
- note removed: "BATTERY"
